Commit message: properly setting finger frames

File: urdf/finger.xacro (robot description, xacro)
@@ -5,5 +5,5 @@
     <parent link="${parent}"/>
     <child link="${name}_link"/>
-    <axis xyz="0 0 1"/>
+    <axis xyz="0 1 0"/>
     <xacro:insert_block name="origin"/>
     <limit effort="50" velocity="10.0" lower="0" upper="3.14" />
@@ -11,10 +11,10 @@
   <link name="${name}_link">
       <inertial>
-          <origin xyz="0.045125 0.00825 0.0275"/>
+          <origin xyz="0.0 0.0 0.0"/>
           <mass value="1.0" />
           <inertia  ixx="1.0" ixy="0.0"  ixz="0.0"  iyy="100.0"  iyz="0.0"  izz="1.0" />
     </inertial>
      <visual>
-        <origin rpy="0 0 0" xyz="0 0 0"/>
+        <origin xyz="0 0.05 0.03" rpy="0 0 0"/>
         <geometry>
             <mesh filename="package://gripper_description/meshes/finger.stl" scale="0.001 0.001 0.001"/>
@@ -22,5 +22,5 @@
      </visual>
      <collision>
-        <origin rpy="0 0 0" xyz="0 0 0"/>
+        <origin  xyz="0 0.05 0.03" rpy="0 0 0"/>
         <geometry>
             <mesh filename="package://gripper_description/meshes/finger.stl" scale="0.001 0.001 0.001"/>

File: urdf/gripper.xacro (robot description, xacro)
@@ -3,7 +3,9 @@
    <xacro:include filename="$(find gripper_description)/urdf/finger.xacro"/>
   <xacro:property name="PI" value="3.1415926535897931"/>
+  <xacro:property name="cos_PI_3" value="0.5"/>
+  <xacro:property name="sin_PI_3" value="0.866"/>
   <link name="gripper_base">
     <inertial>
-      <origin xyz="0.055 0.055 0.055" rpy="0 0 0"/>
+      <origin xyz="0.0 0.0 0.0" rpy="0 0 0"/>
       <mass value="1.0" />
       <inertia  ixx="0.01" ixy="0.0"  ixz="0.0"  iyy="0.01"  iyz="0.0"  izz="0.01" />
@@ -49,15 +51,15 @@
 	name="hand_1"
 	parent="gripper_base">
-	 <origin xyz="0.0 0.0 0.0" rpy="${-PI/2} 0 0"/>
+	 <origin xyz="0.0  -0.03 0.05" rpy="${-PI/2} 0 0"/>
 </xacro:finger>
 <xacro:finger
 	name="hand_2"
 	parent="gripper_base">
-	 <origin xyz="0.0 0.0 0.0" rpy="${-PI/2} 0 ${2*PI/3}"/>
+	 <origin xyz="${0.03*sin_PI_3} ${0.03*cos_PI_3} 0.05" rpy="${-PI/2} 0 ${2*PI/3}"/>
 </xacro:finger>
 <xacro:finger
 	name="hand_3"
 	parent="gripper_base">
-	 <origin xyz="0.0 0.0 0.0" rpy="${-PI/2} 0 ${-2*PI/3}"/>
+	 <origin xyz="${-0.03*sin_PI_3} ${0.03*cos_PI_3} 0.05" rpy="${-PI/2} 0 ${-2*PI/3}"/>
 </xacro:finger>
   <gazebo reference="gripper_base">

Commit message: properly locating gripper_base frame to the attachment point

File: urdf/finger.xacro (robot description, xacro)
@@ -12,6 +12,6 @@
       <inertial>
           <origin xyz="0.0 0.0 0.0"/>
-          <mass value="1.0" />
-          <inertia  ixx="1.0" ixy="0.0"  ixz="0.0"  iyy="100.0"  iyz="0.0"  izz="1.0" />
+          <mass value="0.05" />
+          <inertia  ixx="0.001" ixy="0.0"  ixz="0.0"  iyy="0.001"  iyz="0.0"  izz="0.001" />
     </inertial>
      <visual>

File: urdf/gripper.xacro (robot description, xacro)
@@ -5,5 +5,5 @@
   <xacro:property name="cos_PI_3" value="0.5"/>
   <xacro:property name="sin_PI_3" value="0.866"/>
-  <link name="gripper_base">
+  <link name="gripper_base_down">
     <inertial>
       <origin xyz="0.0 0.0 0.0" rpy="0 0 0"/>
@@ -24,5 +24,5 @@
     </collision>
   </link>
-  <link name="gripper_base_up">
+  <link name="gripper_base">
     <inertial>
       <origin xyz="0.0 0.0 0.0" rpy="0 0 0"/>
@@ -31,5 +31,5 @@
     </inertial>
     <visual>
-      <origin xyz="0.2275 0 -0.06" rpy="${-PI/2} 0 0"/>
+      <origin xyz="0.2275 0 0 " rpy="${-PI/2} 0 0"/>
    	<geometry>
             <mesh filename="package://gripper_description/meshes/gripper_base_up.stl" scale="0.001 0.001 0.001"/>
@@ -37,5 +37,5 @@
     </visual>
     <collision>
-      <origin xyz="0.2275 0 -0.06" rpy="${-PI/2} 0 0"/>
+      <origin xyz="0.2275 0 0" rpy="${-PI/2} 0 0"/>
     <geometry>
             <mesh filename="package://gripper_description/meshes/gripper_base_up.stl" scale="0.001 0.001 0.001"/>
@@ -44,35 +44,23 @@
   </link>
 <joint name="flange" type="fixed">
-		<origin xyz="0 0 0" rpy="0 0 0"/>
+		<origin xyz="0 0 0.06" rpy="0 0 0"/>
 		<parent link="gripper_base"/>
-		<child  link="gripper_base_up"/>
+		<child  link="gripper_base_down"/>
 </joint>
 <xacro:finger
 	name="hand_1"
-	parent="gripper_base">
+	parent="gripper_base_down">
 	 <origin xyz="0.0  -0.03 0.05" rpy="${-PI/2} 0 0"/>
 </xacro:finger>
 <xacro:finger
 	name="hand_2"
-	parent="gripper_base">
+	parent="gripper_base_down">
 	 <origin xyz="${0.03*sin_PI_3} ${0.03*cos_PI_3} 0.05" rpy="${-PI/2} 0 ${2*PI/3}"/>
 </xacro:finger>
 <xacro:finger
 	name="hand_3"
-	parent="gripper_base">
+	parent="gripper_base_down">
 	 <origin xyz="${-0.03*sin_PI_3} ${0.03*cos_PI_3} 0.05" rpy="${-PI/2} 0 ${-2*PI/3}"/>
 </xacro:finger>
-  <gazebo reference="gripper_base">
-    <material>Gazebo/Blue</material>
-  </gazebo>
-  <gazebo reference="gripper_finger_1">
-    <material>Gazebo/Red</material>
-  </gazebo>
-  <gazebo reference="gripper_finger_2">
-    <material>Gazebo/Yellow</material>
-  </gazebo>
-  <gazebo reference="gripper_finger_3">
-    <material>Gazebo/Orange</material>
-  </gazebo>
   <gazebo>
     <plugin name="gazebo_ros_control" filename="libgazebo_ros_control.so">

Commit message: changing gripper axis

File: urdf/finger.xacro (robot description, xacro)
@@ -5,5 +5,5 @@
     <parent link="${parent}"/>
     <child link="${name}_link"/>
-    <axis xyz="0 1 0"/>
+    <axis xyz="0 -1 0"/>
     <xacro:insert_block name="origin"/>
     <limit effort="50" velocity="10.0" lower="0" upper="3.14" />

Commit message: parametrized transmission to have position or effort interface

File: urdf/finger.xacro (robot description, xacro)
@@ -1,5 +1,6 @@
 <?xml version="1.0"?>
 <robot xmlns:xacro="http://ros.org/wiki/xacro">
-<xacro:macro name="finger" params="name parent *origin">
+ <xacro:include filename="$(find gripper_description)/urdf/finger_transmission.xacro" />
+<xacro:macro name="finger" params="name parent transmission_hw_interface *origin">
   <joint name="${name}_joint" type="revolute">
     <parent link="${parent}"/>
@@ -28,4 +29,5 @@
      </collision>
   </link>
+  <xacro:finger_transmission name="${name}" hw_interface="${transmission_hw_interface}" />
 </xacro:macro>
 </robot>

File: urdf/gripper.xacro (robot description, xacro)
@@ -1,5 +1,6 @@
 <?xml version="1.0"?>
 <robot name="gripper" xmlns:xacro="http://ros.org/wiki/xacro">
-   <xacro:include filename="$(find gripper_description)/urdf/finger.xacro"/>
+  <xacro:include filename="$(find gripper_description)/urdf/finger.xacro"/>
+  <xacro:arg name="transmission_hw_interface" default="hardware_interface/EffortJointInterface"/>
   <xacro:property name="PI" value="3.1415926535897931"/>
   <xacro:property name="cos_PI_3" value="0.5"/>
@@ -51,46 +52,19 @@
 <xacro:finger
 	name="hand_1"
-	parent="gripper_base_down">
+	parent="gripper_base_down"
+	transmission_hw_interface="$(arg transmission_hw_interface)">
 	 <origin xyz="0.0  -0.03 0.05" rpy="${-PI/2} 0 0"/>
 </xacro:finger>
 <xacro:finger
 	name="hand_2"
-	parent="gripper_base_down">
+	parent="gripper_base_down"
+	transmission_hw_interface="$(arg transmission_hw_interface)">
 	 <origin xyz="${0.03*sin_PI_3} ${0.03*cos_PI_3} 0.05" rpy="${-PI/2} 0 ${2*PI/3}"/>
 </xacro:finger>
 <xacro:finger
 	name="hand_3"
-	parent="gripper_base_down">
+	parent="gripper_base_down"
+	transmission_hw_interface="$(arg transmission_hw_interface)">
 	 <origin xyz="${-0.03*sin_PI_3} ${0.03*cos_PI_3} 0.05" rpy="${-PI/2} 0 ${-2*PI/3}"/>
 </xacro:finger>
-    <transmission name="hand_1_joint_trans">
-      <type>transmission_interface/SimpleTransmission</type>
-      <joint name="hand_1_joint">
-        <hardwareInterface>hardware_interface/EffortJointInterface</hardwareInterface>
-      </joint>
-      <actuator name="foo_motor_1">
-        <mechanicalReduction>1</mechanicalReduction>
-        <hardwareInterface>hardware_interface/EffortJointInterface</hardwareInterface>
-      </actuator>
-    </transmission>
-    <transmission name="hand_2_joint_trans">
-      <type>transmission_interface/SimpleTransmission</type>
-      <joint name="hand_2_joint">
-        <hardwareInterface>hardware_interface/EffortJointInterface</hardwareInterface>
-      </joint>
-      <actuator name="foo_motor_2">
-        <mechanicalReduction>1</mechanicalReduction>
-        <hardwareInterface>hardware_interface/EffortJointInterface</hardwareInterface>
-      </actuator>
-    </transmission>
-    <transmission name="hand_3_joint_trans">
-      <type>transmission_interface/SimpleTransmission</type>
-      <joint name="hand_3_joint">
-        <hardwareInterface>hardware_interface/EffortJointInterface</hardwareInterface>
-      </joint>
-      <actuator name="foo_motor_3">
-        <mechanicalReduction>1</mechanicalReduction>
-        <hardwareInterface>hardware_interface/EffortJointInterface</hardwareInterface>
-      </actuator>
-    </transmission>
 </robot>

Commit message: setting some contact params

File: urdf/finger.xacro (robot description, xacro)
@@ -30,4 +30,30 @@
   </link>
   <xacro:finger_transmission name="${name}" hw_interface="${transmission_hw_interface}" />
+ <gazebo reference="${name}_link">
+    <collision name="${name}_link_collision">
+      <surface>
+        <friction>
+          <torsional>
+            <coefficient>10.0</coefficient>
+            <use_patch_radius>true</use_patch_radius>
+            <patch_radius>0.05</patch_radius>
+          </torsional>
+        </friction>
+        <contact>
+          <poissons_ratio>0.5</poissons_ratio>
+          <elastic_modulus>1e8</elastic_modulus>
+        </contact>
+      </surface>
+    </collision>
+    <mu1>10</mu1>
+    <mu2>10</mu2>
+    <kp>1000000.0</kp>
+    <kd>10.0</kd>
+    <fdir1>0 0 1</fdir1>
+    <minDepth>0.001</minDepth>
+	    <maxVel>0.0</maxVel>
+    <maxContacts>1</maxContacts>
+    <material>Gazebo/RedBright</material>
+  </gazebo>
 </xacro:macro>
 </robot>

Commit message: created a macro for gripper

File: urdf/finger.xacro (robot description, xacro)
@@ -2,5 +2,7 @@
 <robot xmlns:xacro="http://ros.org/wiki/xacro">
  <xacro:include filename="$(find gripper_description)/urdf/finger_transmission.xacro" />
-<xacro:macro name="finger" params="name parent transmission_hw_interface *origin">
+<xacro:macro name="finger" params="name parent transmission_hw_interface gripper_active *origin">
+<xacro:if value="${gripper_active}">
+  <xacro:finger_transmission name="${name}" hw_interface="${transmission_hw_interface}" />
   <joint name="${name}_joint" type="revolute">
     <parent link="${parent}"/>
@@ -10,4 +12,12 @@
     <limit effort="50" velocity="10.0" lower="0" upper="3.14" />
   </joint>
+</xacro:if>
+<xacro:unless value="${gripper_active}">
+  <joint name="${name}_joint" type="fixed">
+    <parent link="${parent}"/>
+    <child link="${name}_link"/>
+    <xacro:insert_block name="origin"/>
+  </joint>
+</xacro:unless>
   <link name="${name}_link">
       <inertial>
@@ -29,5 +39,4 @@
      </collision>
   </link>
-  <xacro:finger_transmission name="${name}" hw_interface="${transmission_hw_interface}" />
  <gazebo reference="${name}_link">
     <collision name="${name}_link_collision">

File: urdf/gripper.xacro (robot description, xacro)
@@ -1,91 +1,11 @@
 <?xml version="1.0"?>
 <robot name="gripper" xmlns:xacro="http://ros.org/wiki/xacro">
-  <xacro:include filename="$(find gripper_description)/urdf/finger.xacro"/>
-  <xacro:arg name="transmission_hw_interface" default="hardware_interface/EffortJointInterface"/>
-  <xacro:arg name="grasp_plugin" default="true" />
-  <xacro:property name="PI" value="3.1415926535897931"/>
-  <xacro:property name="cos_PI_3" value="0.5"/>
-  <xacro:property name="sin_PI_3" value="0.866"/>
-  <link name="gripper_base_down">
-    <inertial>
-      <origin xyz="0.0 0.0 0.0" rpy="0 0 0"/>
-      <mass value="1.0" />
-      <inertia  ixx="0.01" ixy="0.0"  ixz="0.0"  iyy="0.01"  iyz="0.0"  izz="0.01" />
-    </inertial>
-    <visual>
-      <origin xyz="0 0 0" rpy="${-PI/2} 0 0"/>
-   	<geometry>
-            <mesh filename="package://gripper_description/meshes/gripper_base_down.stl" scale="0.001 0.001 0.001"/>
-        </geometry>
-    </visual>
-    <collision>
-      <origin xyz="0 0 0" rpy="${-PI/2} 0 0"/>
-    <geometry>
-            <mesh filename="package://gripper_description/meshes/gripper_base_down.stl" scale="0.001 0.001 0.001"/>
-        </geometry>
-    </collision>
-  </link>
-  <link name="gripper_base">
-    <visual>
-      <origin xyz="0.2275 0 0 " rpy="${-PI/2} 0 0"/>
-   	<geometry>
-            <mesh filename="package://gripper_description/meshes/gripper_base_up.stl" scale="0.001 0.001 0.001"/>
-        </geometry>
-    </visual>
-    <collision>
-      <origin xyz="0.2275 0 0" rpy="${-PI/2} 0 0"/>
-    <geometry>
-            <mesh filename="package://gripper_description/meshes/gripper_base_up.stl" scale="0.001 0.001 0.001"/>
-        </geometry>
-    </collision>
-  </link>
-<joint name="flange" type="fixed">
-		<origin xyz="0 0 0.06" rpy="0 0 0"/>
-		<parent link="gripper_base"/>
-		<child  link="gripper_base_down"/>
-</joint>
-<joint name="fixed_ee_gripper" type="fixed">
-		<origin xyz="0 0 0.12" rpy="0 0 0"/>
-		<parent link="gripper_base"/>
-		<child  link="ee_gripper"/>
-</joint>
-<link name="ee_gripper"/>
-<xacro:finger
-	name="hand_1"
-	parent="gripper_base_down"
-	transmission_hw_interface="$(arg transmission_hw_interface)">
-	 <origin xyz="0.0  -0.03 0.05" rpy="${-PI/2} 0 0"/>
-</xacro:finger>
-<xacro:finger
-	name="hand_2"
-	parent="gripper_base_down"
-	transmission_hw_interface="$(arg transmission_hw_interface)">
-	 <origin xyz="${0.03*sin_PI_3} ${0.03*cos_PI_3} 0.05" rpy="${-PI/2} 0 ${2*PI/3}"/>
-</xacro:finger>
-<xacro:finger
-	name="hand_3"
-	parent="gripper_base_down"
-	transmission_hw_interface="$(arg transmission_hw_interface)">
-	 <origin xyz="${-0.03*sin_PI_3} ${0.03*cos_PI_3} 0.05" rpy="${-PI/2} 0 ${-2*PI/3}"/>
-</xacro:finger>
-<xacro:if value="$(arg grasp_plugin)">
-	<gazebo>
-	   <plugin name="gazebo_grasp_fix" filename="libgazebo_grasp_fix.so">
-		<arm>
-		   <arm_name>ur5</arm_name>
-		   <palm_link> wrist_3_link  </palm_link>
-		   <gripper_link> hand_1_link </gripper_link>
-		   <gripper_link> hand_2_link </gripper_link>
-		   <gripper_link> hand_3_link </gripper_link>
-		</arm>
-	       <forces_angle_tolerance>100</forces_angle_tolerance>
-	       <update_rate>500</update_rate>
-	       <grip_count_threshold>4</grip_count_threshold>
-	       <max_grip_count>20</max_grip_count>
-	       <release_tolerance>0.01</release_tolerance>
-	       <disable_collisions_on_attach>true</disable_collisions_on_attach>
-	       <contact_topic>__default_topic__</contact_topic>
-	    </plugin>
-	</gazebo>
-</xacro:if>
+		<xacro:include filename="$(find gripper_description)/urdf/gripper.macro.xacro" />
+		<xacro:arg name="transmission_hw_interface" default="hardware_interface/EffortJointInterface" />
+		<xacro:arg name="grasp_plugin" default="false" />
+		<xacro:arg name="gripper_active" default="false" />
+ 		<xacro:gripper
+			transmission_hw_interface="$(arg transmission_hw_interface)"
+			grasp_plugin="$(arg grasp_plugin)"
+			gripper_active="$(arg gripper_active)"/>
 </robot>
