Commit message: added 3d meshes

File: urdf/gripper.xacro (robot description, xacro)
@@ -1,101 +1,64 @@
 <?xml version="1.0"?>
-<robot name="gripper">
+<robot name="gripper" xmlns:xacro="http://ros.org/wiki/xacro">
+   <xacro:include filename="$(find gripper_description)/urdf/finger.xacro"/>
+  <xacro:property name="PI" value="3.1415926535897931"/>
   <link name="gripper_base">
     <inertial>
-      <origin xyz="0.055 0.055 0.055"/>
+      <origin xyz="0.055 0.055 0.055" rpy="0 0 0"/>
       <mass value="1.0" />
       <inertia  ixx="0.01" ixy="0.0"  ixz="0.0"  iyy="0.01"  iyz="0.0"  izz="0.01" />
     </inertial>
     <visual>
-      <origin xyz="0 0 0"/>
-      <geometry>
-        <box size="0.11 0.11 0.11" />
-      </geometry>
+      <origin xyz="0 0 0" rpy="${-PI/2} 0 0"/>
+   	<geometry>
+            <mesh filename="package://gripper_description/meshes/gripper_base_down.stl" scale="0.001 0.001 0.001"/>
+        </geometry>
     </visual>
     <collision>
-      <origin xyz="0 0 0"/>
-      <geometry>
-        <box size="0.11 0.11 0.11" />
-      </geometry>
+      <origin xyz="0 0 0" rpy="${-PI/2} 0 0"/>
+    <geometry>
+            <mesh filename="package://gripper_description/meshes/gripper_base_down.stl" scale="0.001 0.001 0.001"/>
+        </geometry>
     </collision>
   </link>
-  <link name="gripper_finger_1">
+  <link name="gripper_base_up">
     <inertial>
-      <origin xyz="0.045125 0.00825 0.0275"/>
-      <mass value="0.05" />
+      <origin xyz="0.0 0.0 0.0" rpy="0 0 0"/>
+      <mass value="1.0" />
       <inertia  ixx="0.001" ixy="0.0"  ixz="0.0"  iyy="0.001"  iyz="0.0"  izz="0.001" />
     </inertial>
     <visual>
-      <origin xyz="0.015 0 0"/>
-      <geometry>
-        <box size="0.09025 0.0165 0.055" />
-      </geometry>
+      <origin xyz="0.2275 0 -0.06" rpy="${-PI/2} 0 0"/>
+   	<geometry>
+            <mesh filename="package://gripper_description/meshes/gripper_base_up.stl" scale="0.001 0.001 0.001"/>
+        </geometry>
     </visual>
     <collision>
-      <origin xyz="0.015 0 0"/>
-      <geometry>
-        <box size="0.09025 0.0165 0.055" />
-      </geometry>
+      <origin xyz="0.2275 0 -0.06" rpy="${-PI/2} 0 0"/>
+    <geometry>
+            <mesh filename="package://gripper_description/meshes/gripper_base_up.stl" scale="0.001 0.001 0.001"/>
+        </geometry>
     </collision>
   </link>
-  <link name="gripper_finger_2">
-    <inertial>
-      <origin xyz="0.045125 0.00825 0.0275"/>
-      <mass value="0.05" />
-      <inertia  ixx="0.001" ixy="0.0"  ixz="0.0"  iyy="0.001"  iyz="0.0"  izz="0.001" />
-    </inertial>
-    <visual>
-      <origin xyz="0.015 0 0"/>
-      <geometry>
-        <box size="0.09025 0.0165 0.055" />
-      </geometry>
-    </visual>
-    <collision>
-      <origin xyz="0.015 0 0"/>
-      <geometry>
-        <box size="0.09025 0.0165 0.055" />
-      </geometry>
-    </collision>
-  </link>
-  <link name="gripper_finger_3">
-    <inertial>
-      <origin xyz="0.045125 0.00825 0.0275"/>
-      <mass value="0.05" />
-      <inertia  ixx="0.001" ixy="0.0"  ixz="0.0"  iyy="0.001"  iyz="0.0"  izz="0.001" />
-    </inertial>
-    <visual>
-      <origin xyz="0.015 0 0"/>
-      <geometry>
-        <box size="0.09025 0.0165 0.055" />
-      </geometry>
-    </visual>
-    <collision>
-      <origin xyz="0.015 0 0"/>
-      <geometry>
-        <box size="0.09025 0.0165 0.055" />
-      </geometry>
-    </collision>
-  </link>
-  <joint name="hand_1_joint" type="revolute">
-    <parent link="gripper_base"/>
-    <child link="gripper_finger_1"/>
-    <axis xyz="0 0 1"/>
-    <origin xyz="0.015 0.026 0.0835" rpy="0 0 1.047"/>
-    <limit effort="50" velocity="10.0" lower="0" upper="3.14" />
-  </joint>
-  <joint name="hand_2_joint" type="revolute">
-    <parent link="gripper_base"/>
-    <child link="gripper_finger_2"/>
-    <axis xyz="0 0 1"/>
-    <origin xyz="-0.03 0 0.0835" rpy="0 0 3.14"/>
-    <limit effort="50" velocity="10.0" lower="0" upper="3.14" />
-  </joint>
-  <joint name="hand_3_joint" type="revolute">
-    <parent link="gripper_base"/>
-    <child link="gripper_finger_3"/>
-    <axis xyz="0 0 1"/>
-    <origin xyz="0.015 -0.026 0.0835" rpy="0 0 -1.047"/>
-    <limit effort="50" velocity="10.0" lower="0" upper="3.14" />
-  </joint>
+<joint name="flange" type="fixed">
+		<origin xyz="0 0 0" rpy="0 0 0"/>
+		<parent link="gripper_base"/>
+		<child  link="gripper_base_up"/>
+</joint>
+<xacro:finger
+	name="hand_1"
+	parent="gripper_base">
+	 <origin xyz="0.0 0.0 0.0" rpy="${-PI/2} 0 0"/>
+</xacro:finger>
+<xacro:finger
+	name="hand_2"
+	parent="gripper_base">
+	 <origin xyz="0.0 0.0 0.0" rpy="${-PI/2} 0 ${2*PI/3}"/>
+</xacro:finger>
+<xacro:finger
+	name="hand_3"
+	parent="gripper_base">
+	 <origin xyz="0.0 0.0 0.0" rpy="${-PI/2} 0 ${-2*PI/3}"/>
+</xacro:finger>
   <gazebo reference="gripper_base">
     <material>Gazebo/Blue</material>

Commit message: added ee_gripper frame

File: urdf/gripper.xacro (robot description, xacro)
@@ -48,4 +48,10 @@
 		<child  link="gripper_base_down"/>
 </joint>
+<joint name="fixed_ee_gripper" type="fixed">
+		<origin xyz="0 0 0.12" rpy="0 0 0"/>
+		<parent link="gripper_base"/>
+		<child  link="ee_gripper"/>
+</joint>
+<link name="ee_gripper"/>
 <xacro:finger
 	name="hand_1"

Commit message: removing inertia from root joint

File: urdf/gripper.xacro (robot description, xacro)
@@ -25,9 +25,4 @@
   </link>
   <link name="gripper_base">
-    <inertial>
-      <origin xyz="0.0 0.0 0.0" rpy="0 0 0"/>
-      <mass value="1.0" />
-      <inertia  ixx="0.001" ixy="0.0"  ixz="0.0"  iyy="0.001"  iyz="0.0"  izz="0.001" />
-    </inertial>
     <visual>
       <origin xyz="0.2275 0 0 " rpy="${-PI/2} 0 0"/>

Commit message: removed scale factor

File: urdf/gripper.xacro (robot description, xacro)
@@ -4,5 +4,5 @@
 		<xacro:arg name="grasp_plugin" default="true" />
 		<xacro:arg name="gripper_active" default="false" />
-		<xacro:arg name="soft_gripper" default="false" />
+		<xacro:arg name="soft_gripper" default="true" />
 		<xacro:if value="$(arg soft_gripper)">
 			<xacro:include filename="$(find gripper_description)/urdf/soft_gripper.macro.xacro" />

File: urdf/soft_finger.xacro (robot description, xacro)
@@ -35,5 +35,5 @@
 	<origin rpy="0 0 0" xyz="0 0 0" />
 	<geometry>
-	    <mesh filename="package://gripper_description/meshes/soft_gripper_finger1.stl" scale="0.001 0.001 0.001"/>
+	    <mesh filename="package://gripper_description/meshes/soft_gripper_finger1.stl"/>
 	</geometry>
 	</visual>
@@ -41,5 +41,5 @@
 	<origin rpy="0 0 0" xyz="0 0 0" />
 	<geometry>
-	    <mesh filename="package://gripper_description/meshes/soft_gripper_finger1.stl" scale="0.001 0.001 0.001"/>
+	    <mesh filename="package://gripper_description/meshes/soft_gripper_finger1.stl"/>
 	</geometry>
 	</collision>
