Commit message: tuned limits

File: urdf/soft_finger.xacro (robot description, xacro)
@@ -16,5 +16,5 @@
 	    <axis xyz="1 0 0"/>
 	    <xacro:insert_block name="origin"/>
-	    <limit effort="50" velocity="10.0" lower="0" upper="3.14" />
+	    <limit effort="50" velocity="10.0" lower="-0.5" upper="0.3" />
 	  </joint>
 	</xacro:if>
@@ -28,19 +28,19 @@
 	<link name="${name}_link">
 	<inertial>
-	<origin xyz="2.073e-05   1.45286e-03  -1.1049e-03" rpy="0 0 0" />
-	<mass value="0.168" />
-	<inertia ixx="6.69695624e-05" ixy="5.21511788e-09" ixz="-2.74383009e-08" iyy="7.85088161e-05" iyz="5.41105193e-07" izz="1.41819717e-04" />
+		<origin xyz="2.073e-05   1.45286e-03  -1.1049e-03" rpy="0 0 0" />
+		<mass value="0.168" />
+		<inertia ixx="6.69695624e-05" ixy="5.21511788e-09" ixz="-2.74383009e-08" iyy="7.85088161e-05" iyz="5.41105193e-07" izz="1.41819717e-04" />
 	</inertial>
 	<visual>
 	<origin rpy="0 0 0" xyz="0 0 0" />
-	<geometry>
-	    <mesh filename="package://gripper_description/meshes/soft_gripper_finger1.stl"/>
-	</geometry>
+		<geometry>
+		    <mesh filename="package://gripper_description/meshes/soft_gripper_finger1.stl"/>
+		</geometry>
 	</visual>
 	<collision>
 	<origin rpy="0 0 0" xyz="0 0 0" />
-	<geometry>
-	    <mesh filename="package://gripper_description/meshes/soft_gripper_finger1.stl"/>
-	</geometry>
+		<geometry>
+		    <mesh filename="package://gripper_description/meshes/soft_gripper_finger1.stl"/>
+		</geometry>
 	</collision>
 	</link>
@@ -52,18 +52,18 @@
 	<link name="${name}_link2">
 	<visual>
-	<geometry>
-	  <mesh filename="package://gripper_description/meshes/soft_gripper_finger2.stl" />
-	</geometry>
+		<geometry>
+		  <mesh filename="package://gripper_description/meshes/soft_gripper_finger2.stl" />
+		</geometry>
 	<material name="Blue" />
 	</visual>
 	<collision>
-	<geometry>
-	  <mesh filename="package://gripper_description/meshes/soft_gripper_finger2.stl" />
-	</geometry>
+		<geometry>
+		  <mesh filename="package://gripper_description/meshes/soft_gripper_finger2.stl" />
+		</geometry>
 	</collision>
 	<inertial>
 	<origin xyz="2.073e-05   1.45286e-03  -1.1049e-03" rpy="0 0 0" />
-	<mass value="0.168" />
-	<inertia ixx="6.69695624e-05" ixy="5.21511788e-09" ixz="-2.74383009e-08" iyy="7.85088161e-05" iyz="5.41105193e-07" izz="1.41819717e-04" />
+		<mass value="0.168" />
+		<inertia ixx="6.69695624e-05" ixy="5.21511788e-09" ixz="-2.74383009e-08" iyy="7.85088161e-05" iyz="5.41105193e-07" izz="1.41819717e-04" />
 	</inertial>
 	</link>
