Commit message: making hardware interface generic for robotiq gripper

File: gripper_description/urdf/robotiq/robotiq_85_gripper.transmission.xacro (robot description, xacro)
@@ -1,13 +1,13 @@
 <?xml version="1.0"?>
 <robot xmlns:xacro="http://ros.org/wiki/xacro">
-  <xacro:macro name="robotiq_85_gripper_transmission" params="prefix">
+  <xacro:macro name="robotiq_85_gripper_transmission" params="prefix transmission_hw_interface">
         <transmission name="${prefix}robotiq_85_left_knuckle_trans">
             <type>transmission_interface/SimpleTransmission</type>
             <joint name="${prefix}robotiq_85_left_knuckle_joint">
-                <hardwareInterface>hardware_interface/PositionJointInterface</hardwareInterface>
+                <hardwareInterface>${transmission_hw_interface}</hardwareInterface>
             </joint>
             <actuator name="${prefix}robotiq_85_left_knuckle_motor">
                 <mechanicalReduction>1</mechanicalReduction>
-                <hardwareInterface>hardware_interface/PositionJointInterface</hardwareInterface>
+                <hardwareInterface>${transmission_hw_interface}</hardwareInterface>
             </actuator>
         </transmission>

File: gripper_description/urdf/robotiq_gripper.macro.xacro (robot description, xacro)
@@ -323,5 +323,5 @@
 			<material>Gazebo/Grey</material>
 		</gazebo>
-		<xacro:robotiq_85_gripper_transmission prefix="" />
+		<xacro:robotiq_85_gripper_transmission  prefix="" transmission_hw_interface="${transmission_hw_interface}" />
 	<joint name="fixed_ee_gripper" type="fixed">
 			<origin xyz="0 0 0.12" rpy="0 0 0"/>

Commit message: renaming joints for consistency with other grippers

File: gripper_description/urdf/robotiq/robotiq_85_gripper.transmission.xacro (robot description, xacro)
@@ -2,10 +2,10 @@
 <robot xmlns:xacro="http://ros.org/wiki/xacro">
   <xacro:macro name="robotiq_85_gripper_transmission" params="prefix transmission_hw_interface">
-        <transmission name="${prefix}robotiq_85_left_knuckle_trans">
+        <transmission name="${prefix}hand_1_joint_trans">
             <type>transmission_interface/SimpleTransmission</type>
-            <joint name="${prefix}robotiq_85_left_knuckle_joint">
+            <joint name="${prefix}hand_1_joint">
                 <hardwareInterface>${transmission_hw_interface}</hardwareInterface>
             </joint>
-            <actuator name="${prefix}robotiq_85_left_knuckle_motor">
+            <actuator name="${prefix}hand_1_joint_motor">
                 <mechanicalReduction>1</mechanicalReduction>
                 <hardwareInterface>${transmission_hw_interface}</hardwareInterface>
@@ -15,5 +15,5 @@
                 <!-- loading plugin: mimic joints works in gazebo now -->
             <plugin filename="libroboticsgroup_upatras_gazebo_mimic_joint_plugin.so" name="${prefix}mimic_robotiq_85_1">
-                <joint>${prefix}robotiq_85_left_knuckle_joint</joint>
+                <joint>${prefix}hand_1_joint</joint>
                 <mimicJoint>${prefix}robotiq_85_right_knuckle_joint</mimicJoint>
                 <!--multiplier>1.0</multiplier>
@@ -21,5 +21,5 @@
             </plugin>
             <plugin filename="libroboticsgroup_upatras_gazebo_mimic_joint_plugin.so" name="${prefix}mimic_robotiq_85_2">
-                <joint>${prefix}robotiq_85_left_knuckle_joint</joint>
+                <joint>${prefix}hand_1_joint</joint>
                 <mimicJoint>${prefix}robotiq_85_left_inner_knuckle_joint</mimicJoint>
                 <!--multiplier>1.0</multiplier>
@@ -27,5 +27,5 @@
             </plugin>
             <plugin filename="libroboticsgroup_upatras_gazebo_mimic_joint_plugin.so" name="${prefix}mimic_robotiq_85_3">
-                <joint>${prefix}robotiq_85_left_knuckle_joint</joint>
+                <joint>${prefix}hand_1_joint</joint>
                 <mimicJoint>${prefix}robotiq_85_right_inner_knuckle_joint</mimicJoint>
                 <!--multiplier>1.0</multiplier>
@@ -33,5 +33,5 @@
             </plugin>
             <plugin filename="libroboticsgroup_upatras_gazebo_mimic_joint_plugin.so" name="${prefix}mimic_robotiq_85_4">
-                <joint>${prefix}robotiq_85_left_knuckle_joint</joint>
+                <joint>${prefix}hand_1_joint</joint>
                 <mimicJoint>${prefix}robotiq_85_left_finger_tip_joint</mimicJoint>
                 <multiplier>-1.0</multiplier>
@@ -39,5 +39,5 @@
             </plugin>
             <plugin filename="libroboticsgroup_upatras_gazebo_mimic_joint_plugin.so" name="${prefix}mimic_robotiq_85_5">
-                <joint>${prefix}robotiq_85_left_knuckle_joint</joint>
+                <joint>${prefix}hand_1_joint</joint>
                 <mimicJoint>${prefix}robotiq_85_right_finger_tip_joint</mimicJoint>
                 <multiplier>-1.0</multiplier>

File: gripper_description/urdf/robotiq_gripper.macro.xacro (robot description, xacro)
@@ -61,5 +61,5 @@
 			</inertial>
 		</link>
-		<joint name="robotiq_85_left_knuckle_joint" type="revolute">
+		<joint name="hand_1_joint" type="revolute">
 			<parent link="robotiq_85_base_link"/>
 			<child link="robotiq_85_left_knuckle_link"/>
@@ -84,5 +84,5 @@
 			<origin rpy="0.0 0.0 0.0" xyz="0.05490451627 -0.03060114443 0.0"/>
 			<limit lower="-3.14" upper="3.14" velocity="100.0" effort="50"/>
-			<mimic joint="robotiq_85_left_knuckle_joint"/>
+			<mimic joint="hand_1_joint"/>
 			<dynamics damping="100.0" />
 		</joint>
@@ -97,5 +97,5 @@
 		</gazebo>
 		<xacro:mimic_joint_plugin_gazebo name_prefix="{prefix}robotiq_85_right_knuckle_joint"
-			parent_joint="robotiq_85_left_knuckle_joint" mimic_joint="robotiq_85_right_knuckle_joint"
+			parent_joint="hand_1_joint" mimic_joint="robotiq_85_right_knuckle_joint"
 			multiplier="1.0" max_effort="10.0" />
 		<link name="robotiq_85_left_knuckle_link">
@@ -191,8 +191,8 @@
 			<origin xyz="0.06142 0.0127 0" rpy="${pi} 0.0 0.0" />
 			<limit lower="-3.14" upper="3.14" velocity="100.0" effort="0.1"/>
-			<mimic joint="robotiq_85_left_knuckle_joint" offset="0"/>
+			<mimic joint="hand_1_joint" offset="0"/>
 		</joint>
 		<xacro:mimic_joint_plugin_gazebo name_prefix="robotiq_85_left_inner_knuckle_joint"
-			parent_joint="robotiq_85_left_knuckle_joint" mimic_joint="robotiq_85_left_inner_knuckle_joint"
+			parent_joint="hand_1_joint" mimic_joint="robotiq_85_left_inner_knuckle_joint"
 			multiplier="1.0" max_effort="10.0" />
 		<joint name="robotiq_85_right_inner_knuckle_joint" type="continuous">
@@ -202,8 +202,8 @@
 			<origin xyz="0.06142 -0.0127 0" rpy="0 0 0"/>
 			<limit lower="-3.14" upper="3.14" velocity="100.0" effort="0.1"/>
-			<mimic joint="robotiq_85_left_knuckle_joint" offset="0"/>
+			<mimic joint="hand_1_joint" offset="0"/>
 		</joint>
 		<xacro:mimic_joint_plugin_gazebo name_prefix="robotiq_85_right_inner_knuckle_joint"
-			parent_joint="robotiq_85_left_knuckle_joint" mimic_joint="robotiq_85_right_inner_knuckle_joint"
+			parent_joint="hand_1_joint" mimic_joint="robotiq_85_right_inner_knuckle_joint"
 			multiplier="1.0" max_effort="10.0" />
 		<link name="robotiq_85_left_inner_knuckle_link">
@@ -251,8 +251,8 @@
 			<origin xyz="0.04303959807 -0.03759940821 0.0" rpy="0.0 0.0 0.0"/>
 			<limit lower="-3.14" upper="3.14" velocity="100.0" effort="0.1"/>
-			<mimic joint="robotiq_85_left_knuckle_joint" multiplier="-1"/>
+			<mimic joint="hand_1_joint" multiplier="-1"/>
 		</joint>
 		<xacro:mimic_joint_plugin_gazebo name_prefix="robotiq_85_left_finger_tip_joint"
-			parent_joint="robotiq_85_left_knuckle_joint" mimic_joint="robotiq_85_left_finger_tip_joint"
+			parent_joint="hand_1_joint" mimic_joint="robotiq_85_left_finger_tip_joint"
 			multiplier="1.0" max_effort="10.0" />
 		<joint name="robotiq_85_right_finger_tip_joint" type="continuous">
@@ -262,8 +262,8 @@
 			<origin rpy="0.0 0.0 0.0" xyz="0.04303959807 -0.03759940821  0.0"/>
 			<limit lower="-3.14" upper="3.14" velocity="100.0" effort="0.1"/>
-			<mimic joint="robotiq_85_left_knuckle_joint" multiplier="-1"/>
+			<mimic joint="hand_1_joint" multiplier="-1"/>
 		</joint>
 		<xacro:mimic_joint_plugin_gazebo name_prefix="robotiq_85_right_finger_tip_joint"
-			parent_joint="robotiq_85_left_knuckle_joint" mimic_joint="robotiq_85_right_finger_tip_joint"
+			parent_joint="hand_1_joint" mimic_joint="robotiq_85_right_finger_tip_joint"
 			multiplier="1.0" max_effort="10.0" />
 		<link name="robotiq_85_left_finger_tip_link">
@@ -338,6 +338,6 @@
 			   <arm_name>ur5</arm_name>
 			   <palm_link> wrist_3_link  </palm_link>
-			   <gripper_link> hand_1_link </gripper_link>
-			   <gripper_link> hand_2_link </gripper_link>
+			   <gripper_link> robotiq_85_left_finger_link </gripper_link>
+			   <gripper_link> robotiq_85_right_finger_link </gripper_link>
 			</arm>
 		       <forces_angle_tolerance>100</forces_angle_tolerance>
