Commit message: aligned robotiq to ee frame as the other grippers

File: gripper_description/urdf/robotiq_gripper.macro.xacro (robot description, xacro)
@@ -23,5 +23,24 @@
 		</gazebo>
 	</xacro:macro>
-		<link name="gripper_base">
+	  <link name="gripper_base">
+	    <visual>
+	      <origin xyz="0.2275 0 0 " rpy="${-pi/2} 0 0"/>
+	   	<geometry>
+		    <mesh filename="package://gripper_description/meshes/gripper_base_up.stl" scale="0.001 0.001 0.001"/>
+		</geometry>
+	    </visual>
+	    <collision>
+	      <origin xyz="0.2275 0 0" rpy="${-pi/2} 0 0"/>
+	    <geometry>
+		    <mesh filename="package://gripper_description/meshes/gripper_base_up.stl" scale="0.001 0.001 0.001"/>
+		</geometry>
+	    </collision>
+	  </link>
+		<joint name="robotiq_85_base_joint" type="fixed">
+			<parent link="gripper_base"/>
+			<child link="robotiq_85_base_link"/>
+			<origin rpy="0. -${pi/2} 0.0" xyz="0.0 0. 0.0"/>
+		</joint>
+	        <link name="robotiq_85_base_link">
 			<visual>
 				<geometry>
@@ -43,5 +62,5 @@
 		</link>
 		<joint name="robotiq_85_left_knuckle_joint" type="revolute">
-			<parent link="gripper_base"/>
+			<parent link="robotiq_85_base_link"/>
 			<child link="robotiq_85_left_knuckle_link"/>
 			<axis xyz="0 0 1"/>
@@ -60,5 +79,5 @@
 		</gazebo>
 		<joint name="robotiq_85_right_knuckle_joint" type="continuous">
-			<parent link="gripper_base"/>
+			<parent link="robotiq_85_base_link"/>
 			<child link="robotiq_85_right_knuckle_link"/>
 			<axis xyz="0 0 1"/>
@@ -167,5 +186,5 @@
 		</link>
 		<joint name="robotiq_85_left_inner_knuckle_joint" type="continuous">
-			<parent link="gripper_base"/>
+			<parent link="robotiq_85_base_link"/>
 			<child link="robotiq_85_left_inner_knuckle_link"/>
 			<axis xyz="0 0 1"/>
@@ -178,5 +197,5 @@
 			multiplier="1.0" max_effort="10.0" />
 		<joint name="robotiq_85_right_inner_knuckle_joint" type="continuous">
-			<parent link="gripper_base"/>
+			<parent link="robotiq_85_base_link"/>
 			<child link="robotiq_85_right_inner_knuckle_link"/>
 			<axis xyz="0 0 1"/>

Commit message: maxing gripper joint fixed when gripper active = false

File: gripper_description/urdf/robotiq_gripper.macro.xacro (robot description, xacro)
@@ -61,4 +61,12 @@
 			</inertial>
 		</link>
+	<xacro:unless value="${gripper_active}">
+	   <joint name="hand_1_joint" type="fixed">
+    	<parent link="robotiq_85_base_link"/>
+   		 <child link="robotiq_85_left_knuckle_link"/>
+    	 <origin rpy="${pi} 0.0 0.0" xyz="0.05490451627 0.03060114443 0.0"/>
+	   </joint>
+	</xacro:unless>
+	<xacro:if value="${gripper_active}">
 		<joint name="hand_1_joint" type="revolute">
 			<parent link="robotiq_85_base_link"/>
@@ -69,4 +77,5 @@
 			<dynamics damping="100.0" />
 		</joint>
+	</xacro:if>
 		<gazebo reference="robotiq_85_left_knuckle_link">
 			<kp>1000000.0</kp>
@@ -78,13 +87,22 @@
 			<material>Gazebo/Grey</material>
 		</gazebo>
-		<joint name="robotiq_85_right_knuckle_joint" type="continuous">
-			<parent link="robotiq_85_base_link"/>
-			<child link="robotiq_85_right_knuckle_link"/>
-			<axis xyz="0 0 1"/>
-			<origin rpy="0.0 0.0 0.0" xyz="0.05490451627 -0.03060114443 0.0"/>
-			<limit lower="-3.14" upper="3.14" velocity="100.0" effort="50"/>
-			<mimic joint="hand_1_joint"/>
-			<dynamics damping="100.0" />
-		</joint>
+		<xacro:unless value="${gripper_active}">
+		   <joint name="robotiq_85_right_knuckle_joint" type="fixed">
+			<parent link="robotiq_85_base_link"/>
+	   		 <child link="robotiq_85_right_knuckle_link"/>
+			 <origin rpy="0.0 0.0 0.0" xyz="0.05490451627 -0.03060114443 0.0"/>
+		   </joint>
+		</xacro:unless>
+		<xacro:if value="${gripper_active}">
+			<joint name="robotiq_85_right_knuckle_joint" type="continuous">
+				<parent link="robotiq_85_base_link"/>
+				<child link="robotiq_85_right_knuckle_link"/>
+				<axis xyz="0 0 1"/>
+				<origin rpy="0.0 0.0 0.0" xyz="0.05490451627 -0.03060114443 0.0"/>
+				<limit lower="-3.14" upper="3.14" velocity="100.0" effort="50"/>
+				<mimic joint="hand_1_joint"/>
+				<dynamics damping="100.0" />
+			</joint>
+		</xacro:if>
 		<gazebo reference="robotiq_85_right_knuckle_link">
 			<kp>1000000.0</kp>
@@ -185,4 +203,12 @@
 			</inertial>
 		</link>
+		<xacro:unless value="${gripper_active}">
+		   <joint name="robotiq_85_left_inner_knuckle_joint" type="fixed">
+			<parent link="robotiq_85_base_link"/>
+	   		 <child link="robotiq_85_left_inner_knuckle_link"/>
+			<origin xyz="0.06142 0.0127 0" rpy="${pi} 0.0 0.0" />
+		   </joint>
+		</xacro:unless>
+		<xacro:if value="${gripper_active}">
 		<joint name="robotiq_85_left_inner_knuckle_joint" type="continuous">
 			<parent link="robotiq_85_base_link"/>
@@ -193,7 +219,16 @@
 			<mimic joint="hand_1_joint" offset="0"/>
 		</joint>
+		</xacro:if>
 		<xacro:mimic_joint_plugin_gazebo name_prefix="robotiq_85_left_inner_knuckle_joint"
 			parent_joint="hand_1_joint" mimic_joint="robotiq_85_left_inner_knuckle_joint"
 			multiplier="1.0" max_effort="10.0" />
+		<xacro:unless value="${gripper_active}">
+		   <joint name="robotiq_85_right_inner_knuckle_joint" type="fixed">
+			<parent link="robotiq_85_base_link"/>
+	   		 <child link="robotiq_85_right_inner_knuckle_link"/>
+			<origin xyz="0.06142 -0.0127 0" rpy="0 0 0"/>
+		   </joint>
+		</xacro:unless>
+		<xacro:if value="${gripper_active}">
 		<joint name="robotiq_85_right_inner_knuckle_joint" type="continuous">
 			<parent link="robotiq_85_base_link"/>
@@ -204,4 +239,5 @@
 			<mimic joint="hand_1_joint" offset="0"/>
 		</joint>
+		</xacro:if>
 		<xacro:mimic_joint_plugin_gazebo name_prefix="robotiq_85_right_inner_knuckle_joint"
 			parent_joint="hand_1_joint" mimic_joint="robotiq_85_right_inner_knuckle_joint"
@@ -245,15 +281,32 @@
 			</inertial>
 		</link>
-		<joint name="robotiq_85_left_finger_tip_joint" type="continuous">
+		<xacro:unless value="${gripper_active}">
+		   <joint name="robotiq_85_left_finger_tip_joint" type="fixed">
 			<parent link="robotiq_85_left_inner_knuckle_link"/>
-			<child link="robotiq_85_left_finger_tip_link"/>
-			<axis xyz="0 0 1"/>
+	   		 <child link="robotiq_85_left_finger_tip_link"/>
 			<origin xyz="0.04303959807 -0.03759940821 0.0" rpy="0.0 0.0 0.0"/>
-			<limit lower="-3.14" upper="3.14" velocity="100.0" effort="0.1"/>
-			<mimic joint="hand_1_joint" multiplier="-1"/>
-		</joint>
+			</joint>
+		</xacro:unless>
+		<xacro:if value="${gripper_active}">
+			<joint name="robotiq_85_left_finger_tip_joint" type="continuous">
+				<parent link="robotiq_85_left_inner_knuckle_link"/>
+				<child link="robotiq_85_left_finger_tip_link"/>
+				<axis xyz="0 0 1"/>
+				<origin xyz="0.04303959807 -0.03759940821 0.0" rpy="0.0 0.0 0.0"/>
+				<limit lower="-3.14" upper="3.14" velocity="100.0" effort="0.1"/>
+				<mimic joint="hand_1_joint" multiplier="-1"/>
+			</joint>
+		</xacro:if>
 		<xacro:mimic_joint_plugin_gazebo name_prefix="robotiq_85_left_finger_tip_joint"
 			parent_joint="hand_1_joint" mimic_joint="robotiq_85_left_finger_tip_joint"
 			multiplier="1.0" max_effort="10.0" />
+		<xacro:unless value="${gripper_active}">
+		   <joint name="robotiq_85_right_finger_tip_joint" type="fixed">
+			<parent link="robotiq_85_right_inner_knuckle_link"/>
+	   		 <child link="robotiq_85_right_finger_tip_link"/>
+				<origin rpy="0.0 0.0 0.0" xyz="0.04303959807 -0.03759940821  0.0"/>
+			</joint>
+		</xacro:unless>
+		<xacro:if value="${gripper_active}">
 		<joint name="robotiq_85_right_finger_tip_joint" type="continuous">
 			<parent link="robotiq_85_right_inner_knuckle_link"/>
@@ -264,4 +317,5 @@
 			<mimic joint="hand_1_joint" multiplier="-1"/>
 		</joint>
+		</xacro:if>
 		<xacro:mimic_joint_plugin_gazebo name_prefix="robotiq_85_right_finger_tip_joint"
 			parent_joint="hand_1_joint" mimic_joint="robotiq_85_right_finger_tip_joint"
