Commit message: fixing joint with same name as link

File: gripper_description/urdf/gripper.macro.xacro (robot description, xacro)
@@ -39,5 +39,5 @@
 	    </collision>
 	  </link>
-	<joint name="flange" type="fixed">
+	<joint name="flange_fixed_joint" type="fixed">
 			<origin xyz="0 0 0.06" rpy="0 0 0"/>
 			<parent link="gripper_base"/>
